Commit message: joints controller, robot model to fix

File: urdf/man_bot_patrolling.xacro (robot description, xacro)
@@ -165,5 +165,5 @@
     <child link="U_Link"/>
     <axis xyz="0 0 1"/>
-    <limit effort="1000.0" lower="-1.57" upper="1.57" velocity="0.5"/>
+    <limit effort="1000.0" lower="-3.14" upper="3.14" velocity="0.5"/>
     <origin xyz="0 0 0.056"/>
   </joint>

Commit message: robot model with camera fixed and aruco_ros marker_publisher added in launch assignment

File: urdf/man_bot_patrolling.xacro (robot description, xacro)
@@ -33,5 +33,5 @@
       <mass value="0.05"/>
       <origin rpy="0 0 0" xyz="0 0 0"/>
-      <inertia ixx="0.0395416666667" ixy="0" ixz="0" iyy="0.106208333333" iyz="0" izz="0.106208333333"/>
+      <inertia ixx="0.0015416666667" ixy="0" ixz="0" iyy="0.0106208333333" iyz="0" izz="0.0106208333333"/>
     </inertial>
   </link>
@@ -47,5 +47,5 @@
       <mass value="0.1"/>
       <origin rpy="0 0 0" xyz="0 0 0"/>
-      <inertia ixx="0.0395416666667" ixy="0" ixz="0" iyy="0.106208333333" iyz="0" izz="0.106208333333"/>
+      <inertia ixx="0.0015416666667" ixy="0" ixz="0" iyy="0.0106208333333" iyz="0" izz="0.0106208333333"/>
     </inertial>
     <!-- body -->
@@ -79,5 +79,5 @@
     <visual>
       <geometry>
-        <box size="0.015 0.03 0.064"/>
+        <box size="0.015 0.03 0.50"/>
       </geometry>
       <origin rpy="0 0 0" xyz="0 0 0"/>
@@ -87,10 +87,10 @@
       <mass value="0.1"/>
       <origin rpy="0 0 0" xyz="0 0 0"/>
-      <inertia ixx="0.0395416666667" ixy="0" ixz="0" iyy="0.106208333333" iyz="0" izz="0.106208333333"/>
+      <inertia ixx="0.0015416666667" ixy="0" ixz="0" iyy="0.0106208333333" iyz="0" izz="0.0106208333333"/>
     </inertial>
     <!-- body -->
     <collision name="collision_U_link">
       <geometry>
-        <box size="0.015 0.03 0.064"/>
+        <box size="0.015 0.03 0.50"/>
       </geometry>
     </collision>
@@ -147,5 +147,5 @@
       <mass value="0.1"/>
       <origin rpy="0 0 0" xyz="0 0 0"/>
-      <inertia ixx="0.0395416666667" ixy="0" ixz="0" iyy="0.106208333333" iyz="0" izz="0.106208333333"/>
+      <inertia ixx="0.0015416666667" ixy="0" ixz="0" iyy="0.0106208333333" iyz="0" izz="0.0106208333333"/>
     </inertial>
     <!-- body -->
@@ -166,5 +166,5 @@
     <axis xyz="0 0 1"/>
     <limit effort="1000.0" lower="-3.14" upper="3.14" velocity="0.5"/>
-    <origin xyz="0 0 0.056"/>
+    <origin xyz="0 0 0.27"/>
   </joint>
   <joint name="joint_arm_02" type="revolute">
@@ -173,5 +173,5 @@
     <axis xyz="0 1 0"/>
     <limit effort="1000.0" lower="-1.57" upper="1.57" velocity="0.5"/>
-    <origin xyz="0 0 0.036" rpy="0 0 0"/>
+    <origin xyz="0 0 0.25" rpy="0 0 0"/>
   </joint>
   <joint name="servo_mid_to_servo_up" type="fixed">

File: urdf/robot_patrolling_explorer.xacro (robot description, xacro)
@@ -26,14 +26,14 @@
   <link name="robot_base">
     <visual>
-      <origin rpy="1.57 0 3.14" xyz="0.15 -0.117 0"/>
-      <geometry>
-        <mesh scale="0.001 0.001 0.001" filename="package://exprob_robot_patrolling/meshes/robot_chassis.STL"/>
+      <origin rpy="1.57 0 3.14" xyz="0.27 -0.2106 0"/>
+      <geometry>
+        <mesh scale="0.0018 0.0018 0.0018" filename="package://exprob_robot_patrolling/meshes/robot_chassis.STL"/>
       </geometry>
       <material name="red"/>
     </visual>
       <collision>
-      <origin rpy="1.57 0 3.14" xyz="0.15 -0.117 0"/>
-      <geometry>
-        <mesh scale="0.001 0.001 0.001" filename="package://exprob_robot_patrolling/meshes/robot_chassis.STL"/>
+      <origin rpy="1.57 0 3.14" xyz="0.27 -0.2106 0"/>
+      <geometry>
+        <mesh scale="0.0018 0.0018 0.0018" filename="package://exprob_robot_patrolling/meshes/robot_chassis.STL"/>
       </geometry>
     </collision>
@@ -52,5 +52,5 @@
     <parent link="robot_base"/>
     <child link="rbot_base"/>
-    <origin xyz="0 0 0.13787" rpy="0 0 0"/>
+    <origin xyz="0 0 0.242" rpy="0 0 0"/>
   </joint>
 <link name="link_front_right_wheel">
@@ -59,5 +59,5 @@
     <origin rpy="0 1.5707 1.57" xyz="0 0 0"/>
     <geometry>
-      <cylinder length="0.04" radius="0.035"/>
+      <cylinder length="0.07" radius="0.063"/>
     </geometry>
   </collision>
@@ -65,5 +65,5 @@
     <origin rpy="0 1.5707 1.57" xyz="0 0 0"/>
     <geometry>
-      <cylinder length="0.04" radius="0.035"/>
+      <cylinder length="0.07" radius="0.063"/>
     </geometry>
     <material name="grey"/>
@@ -71,5 +71,5 @@
 </link>
 <joint name="joint_front_right_wheel" type="continuous">
-  <origin rpy="0 0 0" xyz="0.07 -0.1 0.035"/>
+  <origin rpy="0 0 0" xyz="0.126 -0.18 0.063"/>
   <child link="link_front_right_wheel" />
   <parent link="robot_base"/>
@@ -83,5 +83,5 @@
     <origin rpy="0 1.5707 1.57" xyz="0 0 0"/>
     <geometry>
-      <cylinder length="0.04" radius="0.035"/>
+      <cylinder length="0.07" radius="0.063"/>
     </geometry>
   </collision>
@@ -89,5 +89,5 @@
     <origin rpy="0 1.5707 1.57" xyz="0 0 0"/>
     <geometry>
-      <cylinder length="0.04" radius="0.035"/>
+      <cylinder length="0.07" radius="0.063"/>
     </geometry>
     <material name="grey"/>
@@ -95,5 +95,5 @@
 </link>
 <joint name="joint_front_left_wheel" type="continuous">
-  <origin rpy="0 0 0" xyz="0.07 0.1 0.035"/>
+  <origin rpy="0 0 0" xyz="0.126 0.18 0.063"/>
   <child link="link_front_left_wheel" />
   <parent link="robot_base"/>
@@ -107,5 +107,5 @@
     <origin rpy="0 1.5707 1.57" xyz="0 0 0"/>
     <geometry>
-      <cylinder length="0.04" radius="0.035"/>
+      <cylinder length="0.07" radius="0.063"/>
     </geometry>
   </collision>
@@ -113,5 +113,5 @@
     <origin rpy="0 1.5707 1.57" xyz="0 0 0"/>
     <geometry>
-      <cylinder length="0.04" radius="0.035"/>
+      <cylinder length="0.07" radius="0.063"/>
     </geometry>
     <material name="grey"/>
@@ -119,5 +119,5 @@
 </link>
 <joint name="joint_rear_right_wheel" type="continuous">
-  <origin rpy="0 0 0" xyz="-0.07 -0.1 0.035"/>
+  <origin rpy="0 0 0" xyz="-0.126 -0.18 0.063"/>
   <child link="link_rear_right_wheel" />
   <parent link="robot_base"/>
@@ -131,5 +131,5 @@
     <origin rpy="0 1.5707 1.57" xyz="0 0 0"/>
     <geometry>
-      <cylinder length="0.04" radius="0.035"/>
+      <cylinder length="0.07" radius="0.063"/>
     </geometry>
   </collision>
@@ -137,5 +137,5 @@
     <origin rpy="0 1.5707 1.57" xyz="0 0 0"/>
     <geometry>
-      <cylinder length="0.04" radius="0.035"/>
+      <cylinder length="0.07" radius="0.063"/>
     </geometry>
     <material name="grey"/>
@@ -143,5 +143,5 @@
 </link>
 <joint name="joint_rear_left_wheel" type="continuous">
-  <origin rpy="0 0 0" xyz="-0.07 0.1 0.035"/>
+  <origin rpy="0 0 0" xyz="-0.126 0.18 0.063"/>
   <child link="link_rear_left_wheel" />
   <parent link="robot_base"/>
@@ -154,5 +154,5 @@
       <origin xyz="0 0 0" rpy="0 0 0" />
       <geometry>
-        <cylinder radius="0.025" length="0.03"/>
+        <cylinder radius="0.045" length="0.05"/>
       </geometry>
       <material name="dark_grey" />
@@ -161,5 +161,5 @@
       <origin xyz="0 0 0" rpy="0 0 0"/>
       <geometry>
-        <cylinder radius="0.025" length="0.03"/>
+        <cylinder radius="0.045" length="0.05"/>
       </geometry>
     </collision>
@@ -167,9 +167,9 @@
       <origin xyz="0 0 0" rpy="0 0 0" />
       <mass value="0.5" />
-      <xacro:cylinder_inertia mass="0.5" r="0.025" l="0.03" />
+      <xacro:cylinder_inertia mass="0.5" r="0.045" l="0.05" />
     </inertial>
   </link>
   <joint name="joint_laser" type="fixed">
-    <origin xyz="0.15 0 0.05" rpy="0 0 0"/>
+    <origin xyz="0.27 0 0.09" rpy="0 0 0"/>
     <parent link="robot_base"/>
     <child link="laser"/>

Commit message: fixed joint of robot's head, arm_joint_03 removed, world generator update

File: urdf/man_bot_patrolling.xacro (robot description, xacro)
@@ -116,11 +116,11 @@
     </collision>
   </link>
-  <link name="servo_up">
-    <visual>
-      <geometry>
-        <cylinder length="0.05" radius="0.015"/>
-      </geometry>
-      <origin rpy="0 0 0" xyz="0 0 0"/>
-      <material name="blue"/>
+  <link name="head_base">
+    <visual>
+      <geometry>
+        <cylinder length="0.05" radius="0.015"/>
+      </geometry>
+      <origin rpy="0 0 0" xyz="0 0 0"/>
+      <material name="light_grey"/>
     </visual>
     <inertial>
@@ -130,5 +130,5 @@
     </inertial>
     <!-- body -->
-    <collision name="collision_servo_up">
+    <collision name="collision_head_base">
       <geometry>
         <cylinder length="0.05" radius="0.015"/>
@@ -175,14 +175,12 @@
     <origin xyz="0 0 0.25" rpy="0 0 0"/>
   </joint>
-  <joint name="servo_mid_to_servo_up" type="fixed">
+  <joint name="servo_mid_to_head_base" type="fixed">
     <parent link="servo_mid"/>
-    <child link="servo_up"/>
+    <child link="head_base"/>
     <origin xyz="0 0 0.0237" rpy="0 1.57 0"/>
   </joint>
-  <joint name="joint_arm_03" type="revolute">
-    <parent link="servo_up"/>
+  <joint name="head_base_camera" type="fixed">
+    <parent link="head_base"/>
     <child link="up_mount"/>
-    <axis xyz="1 0 0"/>
-    <limit effort="1000.0" lower="-1.57" upper="1.57" velocity="0.5"/>
     <origin xyz="-0.028 0 0" rpy="0 -1.57 0"/>
   </joint>
@@ -212,13 +210,3 @@
 	</actuator>
 </transmission>
-<transmission name="joint_arm_03_trans">
-	<type>transmission_interface/SimpleTransmission</type>
-	<joint name="joint_arm_03">
-		<hardwareInterface>hardware_interface/EffortJointInterface</hardwareInterface>
-	</joint>
-	<actuator name="motor3">
-		<hardwareInterface>hardware_interface/EffortJointInterface</hardwareInterface>
-		<mechanicalInterface>1</mechanicalInterface>
-	</actuator>
-</transmission>
 </robot>

Commit message: slam gmapping and fsm working

File: urdf/man_bot_patrolling.xacro (robot description, xacro)
@@ -76,8 +76,8 @@
     </collision>
   </link>
-  <link name="U_Link">
-    <visual>
-      <geometry>
-        <box size="0.015 0.03 0.50"/>
+  <link name="U_Link01">
+    <visual>
+      <geometry>
+        <box size="0.015 0.03 0.25"/>
       </geometry>
       <origin rpy="0 0 0" xyz="0 0 0"/>
@@ -90,10 +90,37 @@
     </inertial>
     <!-- body -->
-    <collision name="collision_U_link">
-      <geometry>
-        <box size="0.015 0.03 0.50"/>
-      </geometry>
-    </collision>
-  </link>
+    <collision name="collision_U_link01">
+      <geometry>
+        <box size="0.015 0.03 0.25"/>
+      </geometry>
+    </collision>
+  </link>
+  <link name="U_Link02">
+    <visual>
+      <geometry>
+        <box size="0.015 0.03 0.25"/>
+      </geometry>
+      <origin rpy="0 0 0" xyz="0 0 -0.125"/>
+      <material name="white"/>
+    </visual>
+    <inertial>
+      <mass value="0.1"/>
+      <origin rpy="0 0 0" xyz="0 0 0"/>
+      <inertia ixx="0.0015416666667" ixy="0" ixz="0" iyy="0.0106208333333" iyz="0" izz="0.0106208333333"/>
+    </inertial>
+    <!-- body -->
+    <collision name="collision_U_link02">
+      <geometry>
+        <box size="0.015 0.03 -0.125"/>
+      </geometry>
+    </collision>
+  </link>
+  <joint name="U_link_extension" type="prismatic">
+    <parent link="U_Link01"/>
+    <child link="U_Link02"/>
+    <axis xyz="0 0 1"/>
+    <limit effort="1000.0" lower="0.0" upper="0.45" velocity="0.5"/>
+    <origin rpy="0 0 0" xyz="0 0 0.125"/>
+  </joint>
   <link name="servo_mid">
     <visual>
@@ -126,5 +153,5 @@
     <inertial>
       <origin xyz="0 0 0" rpy="0 0 0" />
-      <mass value="0.6" />
+      <mass value="0.1" />
       <xacro:cylinder_inertia mass="0.6" r="0.015" l="0.05" />
     </inertial>
@@ -145,5 +172,5 @@
     </visual>
     <inertial>
-      <mass value="0.1"/>
+      <mass value="0.08"/>
       <origin rpy="0 0 0" xyz="0 0 0"/>
       <inertia ixx="0.0015416666667" ixy="0" ixz="0" iyy="0.0106208333333" iyz="0" izz="0.0106208333333"/>
@@ -163,15 +190,15 @@
   <joint name="joint_arm_01" type="revolute">
     <parent link="servo_bottom"/>
-    <child link="U_Link"/>
+    <child link="U_Link01"/>
     <axis xyz="0 0 1"/>
     <limit effort="1000.0" lower="-3.14" upper="3.14" velocity="0.5"/>
-    <origin xyz="0 0 0.27"/>
+    <origin xyz="0 0 0.125"/>
   </joint>
   <joint name="joint_arm_02" type="revolute">
-    <parent link="U_Link"/>
+    <parent link="U_Link02"/>
     <child link="servo_mid"/>
     <axis xyz="0 1 0"/>
     <limit effort="1000.0" lower="-1.57" upper="1.57" velocity="0.5"/>
-    <origin xyz="0 0 0.25" rpy="0 0 0"/>
+    <origin xyz="0 0 0" rpy="0 0 0"/>
   </joint>
   <joint name="servo_mid_to_head_base" type="fixed">
@@ -210,3 +237,13 @@
 	</actuator>
 </transmission>
+<transmission name="joint_link_extension_trans">
+	<type>transmission_interface/SimpleTransmission</type>
+	<joint name="U_link_extension">
+		<hardwareInterface>hardware_interface/EffortJointInterface</hardwareInterface>
+	</joint>
+	<actuator name="motor3">
+		<hardwareInterface>hardware_interface/EffortJointInterface</hardwareInterface>
+		<mechanicalInterface>1</mechanicalInterface>
+	</actuator>
+</transmission>
 </robot>

File: urdf/robot_patrolling_explorer.xacro (robot description, xacro)
@@ -26,5 +26,5 @@
   <link name="robot_base">
     <visual>
-      <origin rpy="1.57 0 3.14" xyz="0.27 -0.2106 0"/>
+      <origin rpy="1.57 0 3.14" xyz="0.27 -0.2106 0.025"/>
       <geometry>
         <mesh scale="0.0018 0.0018 0.0018" filename="package://exprob_robot_patrolling/meshes/robot_chassis.STL"/>
@@ -33,5 +33,5 @@
     </visual>
       <collision>
-      <origin rpy="1.57 0 3.14" xyz="0.27 -0.2106 0"/>
+      <origin rpy="1.57 0 3.14" xyz="0.27 -0.2106 0.025"/>
       <geometry>
         <mesh scale="0.0018 0.0018 0.0018" filename="package://exprob_robot_patrolling/meshes/robot_chassis.STL"/>
@@ -39,6 +39,6 @@
     </collision>
     <inertial>
-      <mass value="5"/>
-      <origin rpy="0 0 0" xyz="0 0 0"/>
+      <mass value="4"/>
+      <origin rpy="0 0 0" xyz="0 0 0.025"/>
       <inertia ixx="0.0395416666667" ixy="0" ixz="0" iyy="0.106208333333" iyz="0" izz="0.106208333333"/>
     </inertial>
@@ -55,9 +55,9 @@
   </joint>
 <link name="link_front_right_wheel">
-  <xacro:default_inertial mass="0.5"/>
+  <xacro:default_inertial mass="0.1"/>
   <collision name="link_front_right_wheel_collision">
     <origin rpy="0 1.5707 1.57" xyz="0 0 0"/>
     <geometry>
-      <cylinder length="0.07" radius="0.063"/>
+      <cylinder length="0.07" radius="0.07"/>
     </geometry>
   </collision>
@@ -65,5 +65,5 @@
     <origin rpy="0 1.5707 1.57" xyz="0 0 0"/>
     <geometry>
-      <cylinder length="0.07" radius="0.063"/>
+      <cylinder length="0.07" radius="0.07"/>
     </geometry>
     <material name="grey"/>
@@ -71,5 +71,5 @@
 </link>
 <joint name="joint_front_right_wheel" type="continuous">
-  <origin rpy="0 0 0" xyz="0.126 -0.18 0.063"/>
+  <origin rpy="0 0 0" xyz="0.126 -0.18 0.07"/>
   <child link="link_front_right_wheel" />
   <parent link="robot_base"/>
@@ -79,9 +79,9 @@
 </joint>
 <link name="link_front_left_wheel">
-  <xacro:default_inertial mass="0.5"/>
+  <xacro:default_inertial mass="0.1"/>
   <collision name="link_front_left_wheel_collision">
     <origin rpy="0 1.5707 1.57" xyz="0 0 0"/>
     <geometry>
-      <cylinder length="0.07" radius="0.063"/>
+      <cylinder length="0.07" radius="0.07"/>
     </geometry>
   </collision>
@@ -89,5 +89,5 @@
     <origin rpy="0 1.5707 1.57" xyz="0 0 0"/>
     <geometry>
-      <cylinder length="0.07" radius="0.063"/>
+      <cylinder length="0.07" radius="0.07"/>
     </geometry>
     <material name="grey"/>
@@ -95,5 +95,5 @@
 </link>
 <joint name="joint_front_left_wheel" type="continuous">
-  <origin rpy="0 0 0" xyz="0.126 0.18 0.063"/>
+  <origin rpy="0 0 0" xyz="0.126 0.18 0.07"/>
   <child link="link_front_left_wheel" />
   <parent link="robot_base"/>
@@ -103,9 +103,9 @@
 </joint>
 <link name="link_rear_right_wheel">
-  <xacro:default_inertial mass="0.5"/>
+  <xacro:default_inertial mass="0.1"/>
   <collision name="link_rear_right_wheel_collision">
     <origin rpy="0 1.5707 1.57" xyz="0 0 0"/>
     <geometry>
-      <cylinder length="0.07" radius="0.063"/>
+      <cylinder length="0.07" radius="0.07"/>
     </geometry>
   </collision>
@@ -113,5 +113,5 @@
     <origin rpy="0 1.5707 1.57" xyz="0 0 0"/>
     <geometry>
-      <cylinder length="0.07" radius="0.063"/>
+      <cylinder length="0.07" radius="0.07"/>
     </geometry>
     <material name="grey"/>
@@ -119,5 +119,5 @@
 </link>
 <joint name="joint_rear_right_wheel" type="continuous">
-  <origin rpy="0 0 0" xyz="-0.126 -0.18 0.063"/>
+  <origin rpy="0 0 0" xyz="-0.126 -0.18 0.07"/>
   <child link="link_rear_right_wheel" />
   <parent link="robot_base"/>
@@ -127,9 +127,9 @@
 </joint>
 <link name="link_rear_left_wheel">
-  <xacro:default_inertial mass="0.5"/>
+  <xacro:default_inertial mass="0.1"/>
   <collision name="link_rear_left_wheel_collision">
     <origin rpy="0 1.5707 1.57" xyz="0 0 0"/>
     <geometry>
-      <cylinder length="0.07" radius="0.063"/>
+      <cylinder length="0.07" radius="0.07"/>
     </geometry>
   </collision>
@@ -137,5 +137,5 @@
     <origin rpy="0 1.5707 1.57" xyz="0 0 0"/>
     <geometry>
-      <cylinder length="0.07" radius="0.063"/>
+      <cylinder length="0.07" radius="0.07"/>
     </geometry>
     <material name="grey"/>
@@ -143,5 +143,5 @@
 </link>
 <joint name="joint_rear_left_wheel" type="continuous">
-  <origin rpy="0 0 0" xyz="-0.126 0.18 0.063"/>
+  <origin rpy="0 0 0" xyz="-0.126 0.18 0.07"/>
   <child link="link_rear_left_wheel" />
   <parent link="robot_base"/>
@@ -175,4 +175,5 @@
     <child link="laser"/>
   </joint>
+<!--
   <transmission name="joint_front_right_wheel_trans">
     <type>transmission_interface/SimpleTransmission</type>
@@ -214,4 +215,4 @@
       <mechanicalInterface>1</mechanicalInterface>
     </actuator>
-  </transmission>
+  </transmission>-->
 </robot>
